File: two_LEDs.kicad_sch (KiCad schematic)
At the start: 4 parts

Commit message: Publish the second iteration of the board
Squashed commit of the following:

commit 03137639306087c590cdda2dc88282cd072a3998
Author: IoT Maestro <iotmaestro@proton.me>
Date:   Wed Sep 20 22:36:39 2023 +0100

    Add JLCPCB PCBA files

commit 878c7d9bf7085809a9e5104ffe31423ea42c8531
Author: IoT Maestro <iotmaestro@proton.me>
Date:   Wed Sep 20 22:35:36 2023 +0100

    Got tired by committing everything one by one...

    Completed revision 2 including placements

commit 69d71586f674b78e869a3471f9a8dc84cc8d366e
Author: IoT Maestro <iotmaestro@proton.me>
Date:   Wed Sep 20 11:49:18 2023 +0100

    Made a few significant changes

     - removed individual channels per region, realistically it'll never be needed
     - added solder pads for all ESP32 pins

commit 97242618a214784a645288727facfb44c62f9649
Author: IoT Maestro <iotmaestro@proton.me>
Date:   Wed Sep 20 07:47:20 2023 +0100

    Assign footprints to components.

commit 45002d8314d0eb1705ebfe038861a6934b1b51b1
Author: IoT Maestro <iotmaestro@proton.me>
Date:   Wed Sep 20 07:42:14 2023 +0100

    Add an XT30 connector for power as well.

commit eac40f851972937518526a0ca66ce5db5aa91d03
Author: IoT Maestro <iotmaestro@proton.me>
Date:   Wed Sep 20 07:24:39 2023 +0100

    Sprinkle a few extra capacitors around for good measures

commit 3b0c2653f8ba452efb0d12ce280c7df2557f22ac
Author: IoT Maestro <iotmaestro@proton.me>
Date:   Wed Sep 20 07:24:15 2023 +0100

    Add .gitignore for backups

commit cc329acc9b2817cd8edc8902f09a11e0c2c65af4
Author: IoT Maestro <iotmaestro@proton.me>
Date:   Wed Sep 20 07:10:53 2023 +0100

    Updated the schematic

     - add 3V3-5V level shifters. This is not necessary but should improve signal integrity.
     - add a series resistor for data lines. Likewise it's not 100% necessary but improves signal integrity and eliminates ringing
Parts:
- C4: footprint Capacitor_SMD:C_0402_1005Metric -> Capacitor_SMD:C_0603_1608Metric; JLCPCB_PART C1525 -> C14663
- D5, D6: value WS2812B -> SK6812-EC20; footprint mapacr:XL-2121RGBC-WS2812B -> mapacr:LED_SK6812-EC20; symbol mapacr:XL-2121RGBC-WS2812B -> mapacr:SK6812-EC20; JLCPCB_PART C5349957 -> C2909058
Changed lines of the file:
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@@
   (junction (at 64.008 32.258) (diameter 0) (color 0 0 0 0)
   )
-  (junction (at 55.88 32.258) (diameter 0) (color 0 0 0 0)
-  )
   (junction (at 48.768 24.638) (diameter 0) (color 0 0 0 0)
   )
+  (junction (at 48.768 47.498) (diameter 0) (color 0 0 0 0)
+  )
   (junction (at 56.642 47.498) (diameter 0) (color 0 0 0 0)
   )
+  (wire (pts (xy 48.768 32.258) (xy 64.008 32.258))
+    (stroke (width 0) (type default))
+  )
   (wire (pts (xy 48.768 47.498) (xy 56.642 47.498))
     (stroke (width 0) (type default))
   )
-  (wire (pts (xy 48.768 32.258) (xy 55.88 32.258))
-    (stroke (width 0) (type default))
-  )
-  (wire (pts (xy 55.88 32.258) (xy 64.008 32.258))
+  (wire (pts (xy 33.02 47.498) (xy 48.768 47.498))
+    (stroke (width 0) (type default))
+  )
+  (wire (pts (xy 78.74 32.258) (xy 64.008 32.258))
+    (stroke (width 0) (type default))
+  )
+  (wire (pts (xy 33.02 24.638) (xy 33.02 47.498))
     (stroke (width 0) (type default))
   )
   (wire (pts (xy 56.642 47.498) (xy 64.008 47.498))
+    (stroke (width 0) (type default))
+  )
+  (wire (pts (xy 78.74 22.86) (xy 78.74 32.258))
     (stroke (width 0) (type default))
   )
@@
       (effects (font (size 1.27 1.27)) (justify left))
     )
-    (property "Footprint" "Capacitor_SMD:C_0402_1005Metric" (at 64.9732 32.258 0)
+    (property "Footprint" "Capacitor_SMD:C_0603_1608Metric" (at 64.9732 32.258 0)
       (effects (font (size 1.27 1.27)) hide)
     )
@@
       (effects (font (size 1.27 1.27)) hide)
     )
-    (property "JLCPCB_PART" "C1525" (at 64.008 28.448 0)
+    (property "JLCPCB_PART" "C14663" (at 64.008 28.448 0)
       (effects (font (size 1.27 1.27)) hide)
     )
@@
       (effects (font (size 1.27 1.27)) (justify left))
     )
-    (property "Footprint" "Capacitor_SMD:C_0402_1005Metric" (at 49.7332 32.258 0)
+    (property "Footprint" "Capacitor_SMD:C_0603_1608Metric" (at 49.7332 32.258 0)
       (effects (font (size 1.27 1.27)) hide)
     )
@@
       (effects (font (size 1.27 1.27)) hide)
     )
-    (property "JLCPCB_PART" "C1525" (at 48.768 28.448 0)
+    (property "JLCPCB_PART" "C14663" (at 48.768 28.448 0)
       (effects (font (size 1.27 1.27)) hide)
     )
@@
     )
   )
-  (symbol (lib_id "mapacr:XL-2121RGBC-WS2812B") (at 48.768 39.878 0) (unit 1)
+  (symbol (lib_id "mapacr:SK6812-EC20") (at 48.768 39.878 0) (unit 1)
     (in_bom yes) (on_board yes) (dnp no)
     (property "Reference" "D5" (at 48.768 51.054 0)
       (effects (font (size 1.27 1.27)))
     )
-    (property "Value" "WS2812B" (at 48.768 52.832 0)
-      (effects (font (size 1.27 1.27)))
-    )
-    (property "Footprint" "mapacr:XL-2121RGBC-WS2812B" (at 50.038 47.498 0)
+    (property "Value" "SK6812-EC20" (at 40.894 48.26 0)
+      (effects (font (size 1.27 1.27)) (justify left top))
+    )
+    (property "Footprint" "mapacr:LED_SK6812-EC20" (at 50.038 47.498 0)
       (effects (font (size 1.27 1.27)) (justify left top) hide)
     )
-    (property "Datasheet" "https://datasheet.lcsc.com/lcsc/2301111010_XINGLIGHT-XL-2121RGBC-WS2812B_C5349957.pdf" (at 51.308 49.403 0)
+    (property "Datasheet" "https://datasheet.lcsc.com/lcsc/2110250930_OPSCO-Optoelectronics-SK6812-EC20_C2909058.pdf" (at 51.308 49.403 0)
       (effects (font (size 1.27 1.27)) (justify left top) hide)
     )
-    (property "JLCPCB_PART" "C5349957" (at 48.768 39.878 0)
+    (property "JLCPCB_PART" "C2909058" (at 57.658 52.578 0)
       (effects (font (size 1.27 1.27)) hide)
     )
@@
     )
   )
-  (symbol (lib_id "power:+5V") (at 55.88 32.258 0) (unit 1)
+  (symbol (lib_id "power:+5V") (at 78.74 22.86 0) (unit 1)
     (in_bom yes) (on_board yes) (dnp no) (fields_autoplaced)
-    (property "Reference" "#PWR03" (at 55.88 36.068 0)
-      (effects (font (size 1.27 1.27)) hide)
-    )
-    (property "Value" "+5V" (at 55.88 28.7561 0)
+    (property "Reference" "#PWR03" (at 78.74 26.67 0)
+      (effects (font (size 1.27 1.27)) hide)
+    )
+    (property "Value" "+5V" (at 78.74 19.3581 0)
       (effects (font (size 1.27 1.27)))
     )
-    (property "Footprint" "" (at 55.88 32.258 0)
-      (effects (font (size 1.27 1.27)) hide)
-    )
-    (property "Datasheet" "" (at 55.88 32.258 0)
+    (property "Footprint" "" (at 78.74 22.86 0)
+      (effects (font (size 1.27 1.27)) hide)
+    )
+    (property "Datasheet" "" (at 78.74 22.86 0)
       (effects (font (size 1.27 1.27)) hide)
     )
@@
     )
   )
-  (symbol (lib_id "power:GND") (at 33.02 24.638 0) (unit 1)
-    (in_bom yes) (on_board yes) (dnp no) (fields_autoplaced)
-    (property "Reference" "#PWR0110" (at 33.02 30.988 0)
-      (effects (font (size 1.27 1.27)) hide)
-    )
-    (property "Value" "GND" (at 33.02 28.7735 0)
-      (effects (font (size 1.27 1.27)))
-    )
-    (property "Footprint" "" (at 33.02 24.638 0)
-      (effects (font (size 1.27 1.27)) hide)
-    )
-    (property "Datasheet" "" (at 33.02 24.638 0)
-      (effects (font (size 1.27 1.27)) hide)
-    )
-    (pin "1")
-    (instances
-      (project "mapacr_budget"
-        (path "/71b974b8-1ba1-4062-b002-6a1a7fefb29b/f52dec1b-c982-41db-b30e-ceff01a37811"
-          (reference "#PWR0110") (unit 1)
-        )
-        (path "/71b974b8-1ba1-4062-b002-6a1a7fefb29b/402cd8cc-f516-424c-85a0-522f37d43c49"
-          (reference "#PWR0111") (unit 1)
-        )
-        (path "/71b974b8-1ba1-4062-b002-6a1a7fefb29b/406a379a-0026-4462-a438-13893326d56e"
-          (reference "#PWR0112") (unit 1)
-        )
-        (path "/71b974b8-1ba1-4062-b002-6a1a7fefb29b/61e8544f-1984-44ab-b3c9-02e9f2cb8537"
-          (reference "#PWR0113") (unit 1)
-        )
-        (path "/71b974b8-1ba1-4062-b002-6a1a7fefb29b/45742699-6e65-4de0-9a9f-deffae99a3e2"
-          (reference "#PWR0114") (unit 1)
-        )
-        (path "/71b974b8-1ba1-4062-b002-6a1a7fefb29b/fd207ae8-3562-48d7-a269-49069aa87ee2"
-          (reference "#PWR0115") (unit 1)
-        )
-        (path "/71b974b8-1ba1-4062-b002-6a1a7fefb29b/efb310ba-6218-4192-a0b7-3542a75ac5f7"
-          (reference "#PWR0116") (unit 1)
-        )
-        (path "/71b974b8-1ba1-4062-b002-6a1a7fefb29b/9ae854d1-0d72-426c-85fa-670aa3eaa4e9"
-          (reference "#PWR0117") (unit 1)
-        )
-        (path "/71b974b8-1ba1-4062-b002-6a1a7fefb29b/4d9fab85-4e20-4961-b776-60f98c0c1888"
-          (reference "#PWR0118") (unit 1)
-        )
-        (path "/71b974b8-1ba1-4062-b002-6a1a7fefb29b/78103047-5bab-49fc-ab7a-b39956314c55"
-          (reference "#PWR0119") (unit 1)
-        )
-        (path "/71b974b8-1ba1-4062-b002-6a1a7fefb29b/a38402cb-9eb1-4ce2-b590-8b6430ce29c2"
-          (reference "#PWR0120") (unit 1)
-        )
-        (path "/71b974b8-1ba1-4062-b002-6a1a7fefb29b/2e8695bb-4c34-48a9-84ee-ec0f63d398a7"
-          (reference "#PWR0121") (unit 1)
-        )
-        (path "/71b974b8-1ba1-4062-b002-6a1a7fefb29b/bd1a698d-6dcf-46f3-96f5-78f3abe20996"
-          (reference "#PWR0122") (unit 1)
-        )
-        (path "/71b974b8-1ba1-4062-b002-6a1a7fefb29b/d92e38d4-b839-483c-918e-0c1e5ec556a2"
-          (reference "#PWR0123") (unit 1)
-        )
-        (path "/71b974b8-1ba1-4062-b002-6a1a7fefb29b/9ac13b8b-e4d7-40cd-ad8c-81a27565fc73"
-          (reference "#PWR0124") (unit 1)
-        )
-        (path "/71b974b8-1ba1-4062-b002-6a1a7fefb29b/afec423d-9fa0-4543-93cb-c92967a72181"
-          (reference "#PWR0125") (unit 1)
-        )
-        (path "/71b974b8-1ba1-4062-b002-6a1a7fefb29b/c59d52a5-9cf2-4713-b9fb-c22002698fe6"
-          (reference "#PWR0126") (unit 1)
-        )
-        (path "/71b974b8-1ba1-4062-b002-6a1a7fefb29b/e6de5ed8-47b0-4eea-80cc-ec626dc5d314"
-          (reference "#PWR0127") (unit 1)
-        )
-      )
-    )
-  )
-  (symbol (lib_id "mapacr:XL-2121RGBC-WS2812B") (at 64.008 39.878 0) (unit 1)
+  (symbol (lib_id "mapacr:SK6812-EC20") (at 64.008 39.878 0) (unit 1)
     (in_bom yes) (on_board yes) (dnp no)
     (property "Reference" "D6" (at 64.008 51.054 0)
       (effects (font (size 1.27 1.27)))
     )
-    (property "Value" "WS2812B" (at 64.008 52.832 0)
-      (effects (font (size 1.27 1.27)))
-    )
-    (property "Footprint" "mapacr:XL-2121RGBC-WS2812B" (at 65.278 47.498 0)
+    (property "Value" "SK6812-EC20" (at 59.69 48.26 0)
+      (effects (font (size 1.27 1.27)) (justify left top))
+    )
+    (property "Footprint" "mapacr:LED_SK6812-EC20" (at 65.278 47.498 0)
       (effects (font (size 1.27 1.27)) (justify left top) hide)
     )
-    (property "Datasheet" "https://datasheet.lcsc.com/lcsc/2301111010_XINGLIGHT-XL-2121RGBC-WS2812B_C5349957.pdf" (at 66.548 49.403 0)
+    (property "Datasheet" "https://datasheet.lcsc.com/lcsc/2110250930_OPSCO-Optoelectronics-SK6812-EC20_C2909058.pdf" (at 66.548 49.403 0)
       (effects (font (size 1.27 1.27)) (justify left top) hide)
     )
-    (property "JLCPCB_PART" "C5349957" (at 64.008 39.878 0)
-      (effects (font (size 1.27 1.27)) hide)
-    )
+    (property "JLCPCB_PART" "C2909058" (at 72.898 52.578 0)
+      (effects (font (size 1.27 1.27)) hide)
+    )
