File: mapacr_budget.kicad_sch (KiCad schematic)
At the start: 52 parts, among them J1 FPC_RIBBON, J2 Barrel_Jack_Switch, J3 FPC_RIBBON, J4 Conn_01x08_Pin, SW1 RESET, SW2 TEST, U1 AMS1117-3.3, U2 ESP32-WROOM-32

Commit message: Publish the second iteration of the board
Squashed commit of the following:

commit 03137639306087c590cdda2dc88282cd072a3998
Author: IoT Maestro <iotmaestro@proton.me>
Date:   Wed Sep 20 22:36:39 2023 +0100

    Add JLCPCB PCBA files

commit 878c7d9bf7085809a9e5104ffe31423ea42c8531
Author: IoT Maestro <iotmaestro@proton.me>
Date:   Wed Sep 20 22:35:36 2023 +0100

    Got tired by committing everything one by one...

    Completed revision 2 including placements

commit 69d71586f674b78e869a3471f9a8dc84cc8d366e
Author: IoT Maestro <iotmaestro@proton.me>
Date:   Wed Sep 20 11:49:18 2023 +0100

    Made a few significant changes

     - removed individual channels per region, realistically it'll never be needed
     - added solder pads for all ESP32 pins

commit 97242618a214784a645288727facfb44c62f9649
Author: IoT Maestro <iotmaestro@proton.me>
Date:   Wed Sep 20 07:47:20 2023 +0100

    Assign footprints to components.

commit 45002d8314d0eb1705ebfe038861a6934b1b51b1
Author: IoT Maestro <iotmaestro@proton.me>
Date:   Wed Sep 20 07:42:14 2023 +0100

    Add an XT30 connector for power as well.

commit eac40f851972937518526a0ca66ce5db5aa91d03
Author: IoT Maestro <iotmaestro@proton.me>
Date:   Wed Sep 20 07:24:39 2023 +0100

    Sprinkle a few extra capacitors around for good measures

commit 3b0c2653f8ba452efb0d12ce280c7df2557f22ac
Author: IoT Maestro <iotmaestro@proton.me>
Date:   Wed Sep 20 07:24:15 2023 +0100

    Add .gitignore for backups

commit cc329acc9b2817cd8edc8902f09a11e0c2c65af4
Author: IoT Maestro <iotmaestro@proton.me>
Date:   Wed Sep 20 07:10:53 2023 +0100

    Updated the schematic

     - add 3V3-5V level shifters. This is not necessary but should improve signal integrity.
     - add a series resistor for data lines. Likewise it's not 100% necessary but improves signal integrity and eliminates ringing
Parts:
- removed J1, J3: FPC_RIBBON, Connector_FFC-FPC:Molex_200528-0300_1x30-1MP_P1.00mm_Horizontal, symbol Connector:Conn_01x30_Socket
- removed JP1, JP10, JP11, JP12, JP13, JP2, JP3, JP4, JP5, JP6, JP7, JP8, JP9: SolderJumper_2_Bridged, Jumper:SolderJumper-2_P1.3mm_Bridged_Pad1.0x1.5mm, symbol Jumper:SolderJumper_2_Bridged
- removed JP14, JP15, JP16, JP17, JP18, JP19, JP20, JP21, JP22, JP23, JP24, JP25, JP26: Jumper_2_Open, Jumper:SolderJumper-2_P1.3mm_Open_Pad1.0x1.5mm, symbol Jumper:Jumper_2_Open
- added C225: 2200u, Capacitor_THT:CP_Radial_D13.0mm_P5.00mm, symbol Device:C_Polarized
- added D7 (x10): SK6812-EC20, mapacr:LED_SK6812-EC20, symbol mapacr:SK6812-EC20
- added J1, J5: Conn_01x18_Socket, mapacr:FPC_1.0K-ES-18PWB, symbol Connector:Conn_01x18_Socket
- added J3: Conn_01x18_Socket, mapacr:FPC_1.0K-ES-18PWB_mechanical_only, symbol Connector:Conn_01x18_Socket
- added Q1: BSS138, Package_TO_SOT_SMD:SOT-23, symbol Transistor_FET:BSS138
- added R19, R5: 470R, Resistor_SMD:R_0402_1005Metric, symbol Device:R
- added R6: 10K, Resistor_SMD:R_0402_1005Metric, symbol Device:R
- added R7: 2K, Resistor_SMD:R_0402_1005Metric, symbol Device:R
- added TP1, TP10, TP11, TP12, TP13, TP14, TP15, TP16, TP17, TP18, TP19, TP2, TP20, TP21, TP22, TP23, TP24, TP25, TP26, TP27, TP28, TP29, TP3, TP30, TP31, TP32, TP33, TP35, TP36, TP4, TP5, TP50, TP51, TP6, TP7, TP8, TP9: TestPoint, mapacr:TestPoint_1.2x3mm, symbol Connector:TestPoint
- added TP34, TP37, TP38, TP39, TP40, TP41, TP42, TP43, TP44, TP45, TP46, TP47, TP48, TP49: TestPoint, TestPoint:TestPoint_Pad_2.5x2.5mm, symbol Connector:TestPoint
- C1, C4: footprint Capacitor_SMD:C_0402_1005Metric -> Capacitor_SMD:C_0603_1608Metric; JLCPCB_PART C1525 -> C14663
- J2: footprint Connector_BarrelJack:BarrelJack_Horizontal -> mapacr:XT30PW-M_and_Barrell_jack
- JP27: value Jumper_2_Bridged -> Jumper_2_Open; footprint Jumper:SolderJumper-2_P1.3mm_Bridged_Pad1.0x1.5mm -> Connector_PinHeader_2.54mm:PinHeader_1x02_P2.54mm_Vertical; symbol Jumper:Jumper_2_Bridged -> Jumper:Jumper_2_Open
- R3: value 10k -> 10K
- R4: value 100K -> 10K; JLCPCB_PART C25741 -> C25744
- SW1, SW2: footprint ts1187:SW_TS-1187A-B-A-B -> mapacr:SW_TS-1187A-B-A-B
Connections:
- net +3V3: now also Q1.1 (G), R6.1, TP35.1
- net +5V: now also J5.11 (Pin_11), J5.12 (Pin_12), J5.13 (Pin_13), J5.14 (Pin_14), J5.5 (Pin_5), J5.6 (Pin_6), J5.7 (Pin_7), J5.8 (Pin_8)
- net +5VA: now also C225.1, J1.11 (Pin_11), J1.12 (Pin_12), J1.13 (Pin_13), J1.14 (Pin_14), J1.5 (Pin_5), J1.6 (Pin_6), J1.7 (Pin_7), J1.8 (Pin_8), R7.1
- net EN: now also TP28.1
- net GND: now also J5.1 (Pin_1), J5.15 (Pin_15), J5.16 (Pin_16), J5.17 (Pin_17), J5.18 (Pin_18), J5.2 (Pin_2), J5.3 (Pin_3), J5.4 (Pin_4)
- net GND1: now also C225.2, J1.1 (Pin_1), J1.15 (Pin_15), J1.16 (Pin_16), J1.17 (Pin_17), J1.18 (Pin_18), J1.2 (Pin_2), J1.3 (Pin_3), J1.4 (Pin_4), TP36.1, TP50.1, TP51.1
- net IO0: now also TP13.1
- net IO2: now also TP11.1
- net JIHOCESKY: now also TP34.1
- net JIHOMORAVSKY: now also TP44.1
- net KARLOVARSKY: now also TP41.1
- net KRALOVEHRADECKY: now also TP49.1
- net LIBERECKY: now also TP39.1
- net MORAVSKOSLEZSKY: now also TP46.1
- net OLOMOUCKY: now also TP47.1
- net PARDUBICKY: now also TP48.1
- net PLZENSKY: now also TP42.1
- net PRAHA: now also J5.10 (Pin_10), J5.9 (Pin_9), R5.1
- net PRAHA_S: now also J1.10 (Pin_10), J1.9 (Pin_9), Q1.3 (D), R7.2; no longer U2.31 (IO19)
- net RX: now also TP10.1
- net STREDOCESKY: now also TP38.1
- net TX: now also TP12.1
- net USTECKY: now also TP40.1
- net VYSOCINA: now also TP43.1
- net ZLINSKY: now also TP45.1
- net eight_LEDs14/DOUT: now also R19.1
- net IO21_TEST: now reaches R4.1, SW2.1, U2.33 (IO21)
- net IO21_TEST: now also TP21.1
- net SDH: now reaches U2.17 (SHD/SD2)
- net SDH: now also TP31.1
- net SWP: now reaches U2.18 (SWP/SD3)
- net SWP: now also TP32.1
- net SCS: now reaches U2.19 (SCS/CMD)
- net SCS: now also TP18.1
- net SCK: now reaches U2.20 (SCK/CLK)
- net SCK: now also TP33.1
- net SDO: now reaches U2.21 (SDO/SD0)
- net SDO: now also TP29.1
- net SDI: now reaches U2.22 (SDI/SD1)
- net SDI: now also TP30.1
- net IO4: now reaches U2.26 (IO4)
- net IO4: now also TP2.1
- net IO22: now reaches U2.36 (IO22)
- net IO22: now also TP16.1
- net IO23: now reaches U2.37 (IO23)
- net IO23: now also TP17.1
- net SENSOR_VP: now reaches U2.4 (SENSOR_VP)
- net SENSOR_VP: now also TP26.1
- net SENSOR_VN: now reaches U2.5 (SENSOR_VN)
- net SENSOR_VN: now also TP27.1
- net IO34: now reaches U2.6 (IO34)
- net IO34: now also TP24.1
- net IO35: now reaches U2.7 (IO35)
- net IO35: now also TP25.1
- net JIHOCESKY_S renamed IO13
- net IO13: now also TP5.1
- net JIHOMORAVSKY_S renamed IO14
- net IO14: now also TP1.1
- net KARLOVARSKY_S renamed IO16
- net IO16: now also TP8.1
- net KRALOVEHRADECKY_S renamed IO32
- net IO32: now also TP22.1
- net LIBERECKY_S renamed IO5
- net IO5: now also TP3.1
- net MORAVSKOSLEZSKY_S renamed IO26
- net IO26: now also TP19.1
- net OLOMOUCKY_S renamed IO25
- net IO25: now also TP6.1
- net PARDUBICKY_S renamed IO33
- net IO33: now also TP23.1
- net PLZENSKY_S renamed IO15
- net IO15: now also TP7.1
- net STREDOCESKY_S renamed IO18
- net IO18: now also TP14.1
- net USTECKY_S renamed IO17
- net IO17: now also TP9.1
- net VYSOCINA_S renamed IO12
- net IO12: now also TP4.1
- net ZLINSKY_S renamed IO27
- net IO27: now also TP20.1
- new net PRAHA_S_3V3: Q1.2 (S), R6.2, TP15.1, U2.31 (IO19)
- new net four_LEDs8/DIN: R5.2, TP37.1
- no-connect marks 15 -> 60
Other:
- note added: "5V-3V3 regulator"
- note added: "ESP32 Dev Module"
- note added: "Logic level shifter"
- note added: "Output headers & solder pads"
- note added: "Power indicators"
- note added: "Power source"
- note added: "Programming header"
- note added: "Spares & back connector"
- note added: "Test PCB controller-map traces"
- moved on the sheet: C1, C2, C3, C4, C5, D210, D211, J4, JP27, JP28, JP29, JP30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

Commit message: Minor adjustments (fixed on-board description, added larger solder pads for power and data)
Parts:
- added TP52: PwrSolderPad, TestPoint:TestPoint_Pad_4.0x4.0mm, symbol Connector:TestPoint
- added TP53: GndSolderPad, TestPoint:TestPoint_Pad_4.0x4.0mm, symbol Connector:TestPoint
- added TP54: DataSolderPad, TestPoint:TestPoint_Pad_2.5x2.5mm, symbol Connector:TestPoint
Connections:
- net +5V: now also TP52.1
- net GND: now also TP53.1
- net PRAHA: now also TP54.1
Changed lines of the file:
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@@
     (stroke (width 0) (type default))
   )
+  (wire (pts (xy 137.16 54.356) (xy 140.208 54.356))
+    (stroke (width 0) (type default))
+  )
   (wire (pts (xy 41.529 89.408) (xy 56.769 89.408))
     (stroke (width 0) (type default))
@@
     (effects (font (size 1.27 1.27)) (justify left bottom))
   )
+  (label "PRAHA" (at 140.208 54.356 0) (fields_autoplaced)
+    (effects (font (size 1.27 1.27)) (justify left bottom))
+  )
   (label "SWP" (at 381.254 239.649 270) (fields_autoplaced)
     (effects (font (size 1.27 1.27)) (justify right bottom))
@@
     (effects (font (size 1.27 1.27)) (justify right bottom))
   )
+  (symbol (lib_id "Connector:TestPoint") (at 156.21 103.124 270) (unit 1)
+    (in_bom yes) (on_board yes) (dnp no) (fields_autoplaced)
+    (property "Reference" "TP53" (at 160.909 102.4803 90)
+      (effects (font (size 1.27 1.27)) (justify left))
+    )
+    (property "Value" "GndSolderPad" (at 160.909 104.4013 90)
+      (effects (font (size 1.27 1.27)) (justify left))
+    )
+    (property "Footprint" "TestPoint:TestPoint_Pad_4.0x4.0mm" (at 156.21 108.204 0)
+      (effects (font (size 1.27 1.27)) hide)
+    )
+    (property "Datasheet" "~" (at 156.21 108.204 0)
+      (effects (font (size 1.27 1.27)) hide)
+    )
+    (pin "1")
+    (instances
+      (project "mapacr_budget"
+        (path "/71b974b8-1ba1-4062-b002-6a1a7fefb29b"
+          (reference "TP53") (unit 1)
+        )
+      )
+    )
+  )
   (symbol (lib_id "mapacr:SK6812-EC20") (at 135.128 124.968 0) (unit 1)
     (in_bom yes) (on_board yes) (dnp no)
@@
     )
   )
+  (symbol (lib_id "Connector:TestPoint") (at 137.16 54.356 90) (unit 1)
+    (in_bom yes) (on_board yes) (dnp no)
+    (property "Reference" "TP54" (at 133.858 50.7111 90)
+      (effects (font (size 1.27 1.27)))
+    )
+    (property "Value" "DataSolderPad" (at 132.842 52.578 90)
+      (effects (font (size 1.27 1.27)))
+    )
+    (property "Footprint" "TestPoint:TestPoint_Pad_2.5x2.5mm" (at 137.16 49.276 0)
+      (effects (font (size 1.27 1.27)) hide)
+    )
+    (property "Datasheet" "~" (at 137.16 49.276 0)
+      (effects (font (size 1.27 1.27)) hide)
+    )
+    (pin "1")
+    (instances
+      (project "mapacr_budget"
+        (path "/71b974b8-1ba1-4062-b002-6a1a7fefb29b"
+          (reference "TP54") (unit 1)
+        )
+      )
+    )
+  )
   (symbol (lib_id "power:GND1") (at 389.89 224.536 0) (unit 1)
     (in_bom yes) (on_board yes) (dnp no) (fields_autoplaced)
@@
         )
       )
+    )
+  )
+  (symbol (lib_id "Connector:TestPoint") (at 152.146 33.782 90) (unit 1)
+    (in_bom yes) (on_board yes) (dnp no) (fields_autoplaced)
+    (property "Reference" "TP52" (at 148.844 30.1371 90)
+      (effects (font (size 1.27 1.27)))
+    )
+    (property "Value" "PwrSolderPad" (at 148.844 32.0581 90)
+      (effects (font (size 1.27 1.27)))
+    )
+    (property "Footprint" "TestPoint:TestPoint_Pad_4.0x4.0mm" (at 152.146 28.702 0)
+      (effects (font (size 1.27 1.27)) hide)
+    )
+    (property "Datasheet" "~" (at 152.146 28.702 0)
+      (effects (font (size 1.27 1.27)) hide)
+    )
+    (pin "1")
+    (instances
+      (project "mapacr_budget"
+        (path "/71b974b8-1ba1-4062-b002-6a1a7fefb29b"
+          (reference "TP52") (unit 1)
+        )
+      )
